Commit message: assignment 6 fixed

File: body0.urdf (robot description, URDF)
Before this commit: robot robot, 5 links, 4 joints
Links:
- added link FrontLeg4, mass 1; collision box size=2.962617745689159 1.3579646896810615 2.16826795597693; visual box size=2.962617745689159 1.3579646896810615 2.16826795597693
- added link FrontLeg5, mass 1; collision box size=1.6654339215792477 1.6042107230838 1.5834378359404093; visual box size=1.6654339215792477 1.6042107230838 1.5834378359404093
- added link FrontLeg6, mass 1; collision box size=1.794698532739853 1.774996647675068 1.1957565270606687; visual box size=1.794698532739853 1.774996647675068 1.1957565270606687
- added link FrontLeg7, mass 1; collision box size=1.8190165381955983 1.5362320215499212 1.3046927612375243; visual box size=1.8190165381955983 1.5362320215499212 1.3046927612375243
- added link FrontLeg8, mass 1; collision box size=1.2847440215373145 1.1601459615422216 2.5027278234596997; visual box size=1.2847440215373145 1.1601459615422216 2.5027278234596997
- added link FrontLeg9, mass 1; collision box size=1.3354112029897136 1.0980368208983833 1.5642072622850025; visual box size=1.3354112029897136 1.0980368208983833 1.5642072622850025
- link BackLeg1: geometry collision box size=1.3115168195904414 1.1197976560829475 1.8607450533826415; visual box size=1.3115168195904414 1.1197976560829475 1.8607450533826415
- link FrontLeg1: geometry collision box size=1.3115168195904414 1.1197976560829475 1.8607450533826415; visual box size=1.3115168195904414 1.1197976560829475 1.8607450533826415
- link FrontLeg2: geometry collision box size=2.9887512410144392 1.0656356799361513 2.5984871306489534; visual box size=2.9887512410144392 1.0656356799361513 2.5984871306489534
- link FrontLeg3: geometry collision box size=2.3450641788730984 1.968895661683963 2.7543711188676667; visual box size=2.3450641788730984 1.968895661683963 2.7543711188676667
- link Torso: geometry collision box size=1.3115168195904414 1.1197976560829475 1.8607450533826415; visual box size=1.3115168195904414 1.1197976560829475 1.8607450533826415
Joints:
- added joint FrontLeg3_FrontLeg4: type revolute, parent FrontLeg3, child FrontLeg4, origin xyz=1.4813088728445796 0.6789823448405308 0 rpy=0 0 0, axis 0 0 1, limit lower=-3.14159 upper=3.14159 effort=0.0 velocity=0.0
- added joint FrontLeg4_FrontLeg5: type revolute, parent FrontLeg4, child FrontLeg5, origin xyz=0.8327169607896239 0.8327169607896239 0 rpy=0 0 0, axis 0 0 1, limit lower=-3.14159 upper=3.14159 effort=0.0 velocity=0.0
- added joint FrontLeg5_FrontLeg6: type revolute, parent FrontLeg5, child FrontLeg6, origin xyz=0.8973492663699265 0.8973492663699265 0 rpy=0 0 0, axis 0 0 1, limit lower=-3.14159 upper=3.14159 effort=0.0 velocity=0.0
- added joint FrontLeg6_FrontLeg7: type revolute, parent FrontLeg6, child FrontLeg7, origin xyz=0.9095082690977991 0.9095082690977991 0 rpy=0 0 0, axis 0 0 1, limit lower=-3.14159 upper=3.14159 effort=0.0 velocity=0.0
- added joint FrontLeg7_FrontLeg8: type revolute, parent FrontLeg7, child FrontLeg8, origin xyz=0.6423720107686572 0.6423720107686572 0 rpy=0 0 0, axis 0 0 1, limit lower=-3.14159 upper=3.14159 effort=0.0 velocity=0.0
- added joint FrontLeg8_FrontLeg9: type revolute, parent FrontLeg8, child FrontLeg9, origin xyz=0.6677056014948568 0.5490184104491916 0 rpy=0 0 0, axis 0 0 1, limit lower=-3.14159 upper=3.14159 effort=0.0 velocity=0.0
- joint FrontLeg1_FrontLeg2: origin xyz=1 0 0 rpy=0 0 0 -> xyz=1.4943756205072196 0.5328178399680756 0 rpy=0 0 0
- joint FrontLeg2_FrontLeg3: origin xyz=1 0 0 rpy=0 0 0 -> xyz=1.1725320894365492 1.1725320894365492 0 rpy=0 0 0
- joint Torso_BackLeg1: origin xyz=-0.5 0 0.5 rpy=0 0 0 -> xyz=-0.6557584097952207 0.5598988280414737 0 rpy=0 0 0
- joint Torso_FrontLeg1: origin xyz=0.5 0 0.5 rpy=0 0 0 -> xyz=0.6557584097952207 0.5598988280414737 0 rpy=0 0 0

File: body1.urdf (robot description, URDF)
Before this commit: robot robot, 9 links, 8 joints
Links:
- added link FrontLeg8, mass 1; collision box size=2.870519406148535 1.1950565320997761 1.9747254705500399; visual box size=2.870519406148535 1.1950565320997761 1.9747254705500399
- added link FrontLeg9, mass 1; collision box size=1.7537515317989147 2.9633331802625085 1.038169752843974; visual box size=1.7537515317989147 2.9633331802625085 1.038169752843974
- link BackLeg1: geometry collision box size=1.7646150559511873 1.882064076760884 1.0057356875289747; visual box size=1.7646150559511873 1.882064076760884 1.0057356875289747
- link FrontLeg1: geometry collision box size=1.7646150559511873 1.882064076760884 1.0057356875289747; visual box size=1.7646150559511873 1.882064076760884 1.0057356875289747
- link FrontLeg2: geometry collision box size=2.3219058460571294 1.6526176271458481 2.557053733540073; visual box size=2.3219058460571294 1.6526176271458481 2.557053733540073
- link FrontLeg3: geometry collision box size=1.8573721917239912 2.4762018760890396 1.5167307574297066; visual box size=1.8573721917239912 2.4762018760890396 1.5167307574297066
- link FrontLeg4: geometry collision box size=1.8688940593868444 1.2603175037905037 1.786883948541412; visual box size=1.8688940593868444 1.2603175037905037 1.786883948541412
- link FrontLeg5: geometry collision box size=1.4502371874289066 1.72945595677036 1.3275242840109511; visual box size=1.4502371874289066 1.72945595677036 1.3275242840109511
- link FrontLeg6: geometry collision box size=1.5238882073992566 2.707913573088801 1.6117715230562677; visual box size=1.5238882073992566 2.707913573088801 1.6117715230562677
- link FrontLeg7: geometry collision box size=2.8971748565024837 1.2765618825493164 2.1701518996999543; visual box size=2.8971748565024837 1.2765618825493164 2.1701518996999543
- link Torso: geometry collision box size=1.7646150559511873 1.882064076760884 1.0057356875289747; visual box size=1.7646150559511873 1.882064076760884 1.0057356875289747
Joints:
- added joint FrontLeg7_FrontLeg8: type revolute, parent FrontLeg7, child FrontLeg8, origin xyz=1.4352597030742675 0.5975282660498881 0 rpy=0 0 0, axis 0 0 1, limit lower=-3.14159 upper=3.14159 effort=0.0 velocity=0.0
- added joint FrontLeg8_FrontLeg9: type revolute, parent FrontLeg8, child FrontLeg9, origin xyz=0.8768757658994574 1.4816665901312542 0 rpy=0 0 0, axis 0 0 1, limit lower=-3.14159 upper=3.14159 effort=0.0 velocity=0.0
- joint FrontLeg1_FrontLeg2: origin xyz=1 0 0 rpy=0 0 0 -> xyz=1.1609529230285647 1.1609529230285647 0 rpy=0 0 0
- joint FrontLeg2_FrontLeg3: origin xyz=1 0 0 rpy=0 0 0 -> xyz=0.9286860958619956 0.9286860958619956 0 rpy=0 0 0
- joint FrontLeg3_FrontLeg4: origin xyz=1 0 0 rpy=0 0 0 -> xyz=0.9344470296934222 0.9344470296934222 0 rpy=0 0 0
- joint FrontLeg4_FrontLeg5: origin xyz=1 0 0 rpy=0 0 0 -> xyz=0.7251185937144533 0.7251185937144533 0 rpy=0 0 0
- joint FrontLeg5_FrontLeg6: origin xyz=1 0 0 rpy=0 0 0 -> xyz=0.7619441036996283 0.7619441036996283 0 rpy=0 0 0
- joint FrontLeg6_FrontLeg7: origin xyz=1 0 0 rpy=0 0 0 -> xyz=1.4485874282512419 1.4485874282512419 0 rpy=0 0 0
- joint Torso_BackLeg1: origin xyz=-0.5 0 0.5 rpy=0 0 0 -> xyz=-0.8823075279755936 0.941032038380442 0 rpy=0 0 0
- joint Torso_FrontLeg1: origin xyz=0.5 0 0.5 rpy=0 0 0 -> xyz=0.8823075279755936 0.941032038380442 0 rpy=0 0 0

Commit message: assignment 7 done

File: body0.urdf (robot description, URDF)
Before this commit: robot robot, 11 links, 10 joints
Links:
- removed link BackLeg1
- removed link FrontLeg1
- removed link FrontLeg2
- removed link FrontLeg3
- removed link FrontLeg4
- removed link FrontLeg5
- removed link FrontLeg6
- removed link FrontLeg7
- removed link FrontLeg8
- removed link FrontLeg9
- removed link Torso
- added link Segment0, mass 1; collision box size=1.2227375255694746 1.4188719473436937 1.2112965306504988; visual box size=1.2227375255694746 1.4188719473436937 1.2112965306504988
- added link Segment1, mass 1; collision box size=1.1796646338788919 1.1917008896392958 1.540291639080816; visual box size=1.1796646338788919 1.1917008896392958 1.540291639080816
- added link Segment10, mass 1; collision box size=1.290590291403253 1.3035977646198489 1.2338984329967464; visual box size=1.290590291403253 1.3035977646198489 1.2338984329967464
- added link Segment2, mass 1; collision box size=1.3413495902122827 1.3607716994443886 1.2405317880562934; visual box size=1.3413495902122827 1.3607716994443886 1.2405317880562934
- added link Segment3, mass 1; collision box size=1.7214737315209923 1.7973719322892951 1.7591130042026528; visual box size=1.7214737315209923 1.7973719322892951 1.7591130042026528
- added link Segment4, mass 1; collision box size=1.2239730051154467 1.8646200518854943 1.309186736159782; visual box size=1.2239730051154467 1.8646200518854943 1.309186736159782
- added link Segment5, mass 1; collision box size=1.6221599255763453 1.0249748752689742 1.4451971879395829; visual box size=1.6221599255763453 1.0249748752689742 1.4451971879395829
- added link Segment6, mass 1; collision box size=1.3991375041931007 1.8715813485861323 1.55581639428304; visual box size=1.3991375041931007 1.8715813485861323 1.55581639428304
- added link Segment7, mass 1; collision box size=1.367502356068552 1.276323223477382 1.3348532585776751; visual box size=1.367502356068552 1.276323223477382 1.3348532585776751
- added link Segment8, mass 1; collision box size=1.3687730744833133 1.3241973308733315 1.4868247272806725; visual box size=1.3687730744833133 1.3241973308733315 1.4868247272806725
- added link Segment9, mass 1; collision box size=1.8453801820070015 1.4671619546249408 1.4252479013488422; visual box size=1.8453801820070015 1.4671619546249408 1.4252479013488422
Joints:
- removed joint FrontLeg1_FrontLeg2
- removed joint FrontLeg2_FrontLeg3
- removed joint FrontLeg3_FrontLeg4
- removed joint FrontLeg4_FrontLeg5
- removed joint FrontLeg5_FrontLeg6
- removed joint FrontLeg6_FrontLeg7
- removed joint FrontLeg7_FrontLeg8
- removed joint FrontLeg8_FrontLeg9
- removed joint Torso_BackLeg1
- removed joint Torso_FrontLeg1
- added joint Segment0_Segment1: type revolute, parent Segment0, child Segment1, origin xyz=-0.6113687627847373 0.7094359736718469 7.468304667625675 rpy=0 0 0, axis 0 1 1, limit lower=-3.14159 upper=3.14159 effort=0.0 velocity=0.0
- added joint Segment0_Segment2: type revolute, parent Segment0, child Segment2, origin xyz=-0.6113687627847373 -0.7094359736718469 7.468304667625675 rpy=0 0 0, axis 0 1 1, limit lower=-3.14159 upper=3.14159 effort=0.0 velocity=0.0
- added joint Segment1_Segment3: type revolute, parent Segment1, child Segment3, origin xyz=0.0 0.0 -1.540291639080816 rpy=0 0 0, axis 0 1 1, limit lower=-3.14159 upper=3.14159 effort=0.0 velocity=0.0
- added joint Segment2_Segment4: type revolute, parent Segment2, child Segment4, origin xyz=0.6803858497221943 -0.6803858497221943 -1.2405317880562934 rpy=0 0 0, axis 0 1 1, limit lower=-3.14159 upper=3.14159 effort=0.0 velocity=0.0
- added joint Segment3_Segment5: type revolute, parent Segment3, child Segment5, origin xyz=0.8986859661446476 0.0 -1.7591130042026528 rpy=0 0 0, axis 0 1 1, limit lower=-3.14159 upper=3.14159 effort=0.0 velocity=0.0
- added joint Segment4_Segment6: type revolute, parent Segment4, child Segment6, origin xyz=0.9323100259427471 -0.9323100259427471 -1.309186736159782 rpy=0 0 0, axis 0 1 1, limit lower=-3.14159 upper=3.14159 effort=0.0 velocity=0.0
- added joint Segment5_Segment7: type revolute, parent Segment5, child Segment7, origin xyz=0.0 0.5124874376344871 -1.4451971879395829 rpy=0 0 0, axis 0 1 1, limit lower=-3.14159 upper=3.14159 effort=0.0 velocity=0.0
- added joint Segment6_Segment8: type revolute, parent Segment6, child Segment8, origin xyz=0.0 -0.0 -1.55581639428304 rpy=0 0 0, axis 0 1 1, limit lower=-3.14159 upper=3.14159 effort=0.0 velocity=0.0
- added joint Segment7_Segment9: type revolute, parent Segment7, child Segment9, origin xyz=0.638161611738691 0.0 -1.3348532585776751 rpy=0 0 0, axis 0 1 1, limit lower=-3.14159 upper=3.14159 effort=0.0 velocity=0.0
- added joint Segment8_Segment10: type revolute, parent Segment8, child Segment10, origin xyz=0.0 -0.6620986654366657 -1.4868247272806725 rpy=0 0 0, axis 0 1 1, limit lower=-3.14159 upper=3.14159 effort=0.0 velocity=0.0

File: body1.urdf (robot description, URDF)
Before this commit: robot robot, 11 links, 10 joints
Links:
- removed link BackLeg1
- removed link FrontLeg1
- removed link FrontLeg2
- removed link FrontLeg3
- removed link FrontLeg4
- removed link FrontLeg5
- removed link FrontLeg6
- removed link FrontLeg7
- removed link FrontLeg8
- removed link FrontLeg9
- removed link Torso
- added link Segment0, mass 1; collision box size=1.4567813940615606 1.134319541754019 1.0402946828618573; visual box size=1.4567813940615606 1.134319541754019 1.0402946828618573
- added link Segment1, mass 1; collision box size=1.0594005927001737 1.446247328839966 1.2477160651979822; visual box size=1.0594005927001737 1.446247328839966 1.2477160651979822
- added link Segment10, mass 1; collision box size=1.5782526062587368 1.8395111143693716 1.4668858618514076; visual box size=1.5782526062587368 1.8395111143693716 1.4668858618514076
- added link Segment2, mass 1; collision box size=1.4621088343765096 1.0307217331400897 1.337519212621152; visual box size=1.4621088343765096 1.0307217331400897 1.337519212621152
- added link Segment3, mass 1; collision box size=1.3908571380914052 1.2750903205521562 1.4918596283080174; visual box size=1.3908571380914052 1.2750903205521562 1.4918596283080174
- added link Segment4, mass 1; collision box size=1.2842869455144608 1.0888818429284006 1.3664019313647442; visual box size=1.2842869455144608 1.0888818429284006 1.3664019313647442
- added link Segment5, mass 1; collision box size=1.2056649758596023 1.1535334918766293 1.7063866500876015; visual box size=1.2056649758596023 1.1535334918766293 1.7063866500876015
- added link Segment6, mass 1; collision box size=1.4777728405296882 1.823396369277606 1.3486769278205815; visual box size=1.4777728405296882 1.823396369277606 1.3486769278205815
- added link Segment7, mass 1; collision box size=1.4482535927204407 1.0765523246833761 1.7411496061345488; visual box size=1.4482535927204407 1.0765523246833761 1.7411496061345488
- added link Segment8, mass 1; collision box size=1.2323309994594827 1.4776543173318508 1.0224077527948014; visual box size=1.2323309994594827 1.4776543173318508 1.0224077527948014
- added link Segment9, mass 1; collision box size=1.4675336025307968 1.2497792476334115 1.1308954641132996; visual box size=1.4675336025307968 1.2497792476334115 1.1308954641132996
Joints:
- removed joint FrontLeg1_FrontLeg2
- removed joint FrontLeg2_FrontLeg3
- removed joint FrontLeg3_FrontLeg4
- removed joint FrontLeg4_FrontLeg5
- removed joint FrontLeg5_FrontLeg6
- removed joint FrontLeg6_FrontLeg7
- removed joint FrontLeg7_FrontLeg8
- removed joint FrontLeg8_FrontLeg9
- removed joint Torso_BackLeg1
- removed joint Torso_FrontLeg1
- added joint Segment0_Segment1: type revolute, parent Segment0, child Segment1, origin xyz=-0.7283906970307803 0.5671597708770095 7.190023220862533 rpy=0 0 0, axis 0 1 1, limit lower=-3.14159 upper=3.14159 effort=0.0 velocity=0.0
- added joint Segment0_Segment2: type revolute, parent Segment0, child Segment2, origin xyz=-0.7283906970307803 -0.5671597708770095 7.190023220862533 rpy=0 0 0, axis 0 1 1, limit lower=-3.14159 upper=3.14159 effort=0.0 velocity=0.0
- added joint Segment1_Segment3: type revolute, parent Segment1, child Segment3, origin xyz=0.0 0.0 -1.2477160651979822 rpy=0 0 0, axis 0 1 1, limit lower=-3.14159 upper=3.14159 effort=0.0 velocity=0.0
- added joint Segment2_Segment4: type revolute, parent Segment2, child Segment4, origin xyz=0.5153608665700449 -0.0 -1.337519212621152 rpy=0 0 0, axis 0 1 1, limit lower=-3.14159 upper=3.14159 effort=0.0 velocity=0.0
- added joint Segment3_Segment5: type revolute, parent Segment3, child Segment5, origin xyz=0.6375451602760781 0.0 -1.4918596283080174 rpy=0 0 0, axis 0 1 1, limit lower=-3.14159 upper=3.14159 effort=0.0 velocity=0.0
- added joint Segment4_Segment6: type revolute, parent Segment4, child Segment6, origin xyz=0.5444409214642003 -0.5444409214642003 -1.3664019313647442 rpy=0 0 0, axis 0 1 1, limit lower=-3.14159 upper=3.14159 effort=0.0 velocity=0.0
- added joint Segment5_Segment7: type revolute, parent Segment5, child Segment7, origin xyz=0.5767667459383147 0.5767667459383147 -1.7063866500876015 rpy=0 0 0, axis 0 1 1, limit lower=-3.14159 upper=3.14159 effort=0.0 velocity=0.0
- added joint Segment6_Segment8: type revolute, parent Segment6, child Segment8, origin xyz=0.911698184638803 -0.0 -1.3486769278205815 rpy=0 0 0, axis 0 1 1, limit lower=-3.14159 upper=3.14159 effort=0.0 velocity=0.0
- added joint Segment7_Segment9: type revolute, parent Segment7, child Segment9, origin xyz=0.0 0.0 -1.7411496061345488 rpy=0 0 0, axis 0 1 1, limit lower=-3.14159 upper=3.14159 effort=0.0 velocity=0.0
- added joint Segment8_Segment10: type revolute, parent Segment8, child Segment10, origin xyz=0.7388271586659254 -0.7388271586659254 -1.0224077527948014 rpy=0 0 0, axis 0 1 1, limit lower=-3.14159 upper=3.14159 effort=0.0 velocity=0.0
